File: micro-amps.kicad_pcb (KiCad board)
At the start: 2 copper layers, 60.7 x 39.1 mm, 21 parts, among them J1 Conn_01x04_Pin, J2 Conn_01x01_Socket, J3 Conn_02x04_Odd_Even, J4 Conn_01x01_Socket, J5 Conn_01x01_Socket, J6 Conn_01x01_Socket, SW1 SW_Slide_DPDT, U1 OPA197xDBV

Commit message: Dual OPAMP stage
Parts:
- removed the J1 at (140.8, 87.6)
- added C3: 10p, Capacitor_SMD:C_0603_1608Metric_Pad1.08x0.95mm_HandSolder, F.Cu at (125.9, 80.9)
- added R10: 10k, Resistor_SMD:R_0603_1608Metric_Pad0.98x0.95mm_HandSolder, F.Cu at (123.2, 79.8)
- added R4: 47k, Resistor_SMD:R_0603_1608Metric_Pad0.98x0.95mm_HandSolder, F.Cu at (125.1, 78.2)
- added R5: 43k, Resistor_SMD:R_0603_1608Metric_Pad0.98x0.95mm_HandSolder, F.Cu at (127.5, 80.9)
- R2: value 56k -> 47k
- R9: renamed from R7; value 1k -> 10k
- U1: value OPA197xDBV -> OPA2197xDGK; footprint Package_TO_SOT_SMD:SOT-23-5_HandSoldering -> Package_SO:VSSOP-8_3x3mm_P0.65mm
- moved R2 6.26 mm to (123.2, 89.4), turned to 0 degrees
- moved C1 4.05 mm to (126.1, 84.6)
- moved R9 3.63 mm to (120.5, 86.9), turned to -90 degrees
- moved R1 3.49 mm to (120.5, 83.4), turned to 90 degrees
- moved R3 3.30 mm to (125.7, 88.5), turned to 90 degrees
- moved U1 2.26 mm to (123.2, 83.8)
- moved C2 0.93 mm to (123.2, 87.9)
- renumbered J2 to J1, J4 to J2, J5 to J4, J6 to J5, R4 to R6, R5 to R7, R6 to R8
Connections:
- C2 pad 1: Net-(J4-Pin_1) -> Net-(U1A-+)
- C2 pad 2: Net-(U1--) -> Net-(U1B--)
- J2 pad 1: Net-(J4-Pin_1) -> Net-(J2-Pin_1)
- R1 pad 1: Net-(U1-+) -> Net-(U1B-+)
- R2 pad 1: Net-(U1--) -> Net-(U1B--)
- R3 pad 2: Net-(J4-Pin_1) -> Net-(U1A-+)
- R9 pad 2: Net-(U1--) -> Net-(U1B--)
- U1 pad 1: Net-(J4-Pin_1) -> Net-(J2-Pin_1)
- U1 pad 2: -12V -> Net-(U1A--)
- U1 pad 3: Net-(U1-+) -> Net-(U1A-+)
- U1 pad 4: Net-(U1--) -> -12V
- U1 pad 5: +12V -> Net-(U1B-+)
Routing:
- net Net-(J4-Pin_1): track 37.9 -> 0.00 mm
- net Net-(J2-Pin_1): track 0.00 -> 34.0 mm
- net Net-(BT2--): track 23.1 -> 14.3 mm
- net Net-(U1--): track 8.50 -> 0.00 mm
- net Net-(U1A-+): track 0.00 -> 8.46 mm
- net Net-(BT1-+): track 25.2 -> 18.3 mm
- net Net-(U1A--): track 0.00 -> 5.62 mm
- net Net-(U1B--): track 0.00 -> 5.57 mm
- net -12V: track 9.28 -> 13.1 mm, vias 0 -> 2
- net Net-(U1B-+): track 0.00 -> 2.97 mm
- net Net-(U1-+): track 2.55 -> 0.00 mm
- net Net-(R4-Pad2): track 0.00 -> 2.38 mm
- net Net-(J1-Pin_1): track 34.4 -> 35.0 mm
