File: micro-amps.kicad_pcb (KiCad board)
At the start: 2 copper layers, 60.7 x 39.1 mm, 21 parts, among them J1 Conn_01x04_Pin, J2 Conn_01x01_Socket, J3 Conn_02x04_Odd_Even, J4 Conn_01x01_Socket, J5 Conn_01x01_Socket, J6 Conn_01x01_Socket, SW1 SW_Slide_DPDT, U1 OPA197xDBV

Commit message: Optimize layout
Parts:
- removed the J1 at (140.8, 87.6)
- moved C2 2.31 mm to (125.6, 85.7)
- moved J2 1.77 mm to (118.4, 87.6)
- moved R4 1.77 mm to (109.2, 85.1)
- moved R5 1.77 mm to (109.2, 82.5)
- moved R6 1.77 mm to (109.2, 80.0)
- moved SW1 1.77 mm to (135.8, 82.0)
- moved R3 1.76 mm to (124.6, 87.4)
- moved R1 1.50 mm to (122.7, 80.0)
- moved R2 1.50 mm to (123.6, 83.2)
- moved U1 1.50 mm to (126.4, 82.4)
- moved C1 1.50 mm to (129.5, 81.0)
- moved R7 1.50 mm to (121.9, 83.2)
- moved BT2 0.25 mm to (111.6, 69.6)
- renumbered J2 to J1, J3 to J2, J4 to J3, J5 to J4, J6 to J5
Routing:
- net Net-(BT2--): track 23.1 -> 15.8 mm
- net Net-(BT1-+): track 25.2 -> 20.1 mm
- net Net-(J3-Pin_1): track 37.9 -> 34.0 mm
- net Net-(U1--): track 8.50 -> 6.84 mm
- net Net-(J1-Pin_1): track 34.4 -> 35.8 mm
- net Net-(R2-Pad2): track 1.99 -> 3.24 mm
Other:
- board text added: "±1.2 mA"
- board text added: "±12 µA"
- board text added: "±120 mA"
- board text removed: "GND"
- board text removed: "±1 mA"
- board text removed: "±10 µA"
- board text removed: "±100 mA"

Commit message: Refine things
Routing:
- net Net-(J3-Pin_1): track 34.0 -> 31.9 mm
