File: micro-amps.kicad_sch (KiCad schematic)
At the start: 21 parts, among them J1 Conn_01x04_Pin, J2 Conn_01x01_Socket, J3 Conn_02x04_Odd_Even, J4 Conn_01x01_Socket, J5 Conn_01x01_Socket, J6 Conn_01x01_Socket, SW1 SW_Slide_DPDT, U1 OPA197xDBV

Commit message: Optimize layout
Parts:
- removed J1: Conn_01x04_Pin, Connector_PinHeader_2.54mm:PinHeader_1x04_P2.54mm_Vertical, symbol Connector:Conn_01x04_Pin
- renumbered J2 to J1, J3 to J2, J4 to J3, J5 to J4, J6 to J5
Other:
- moved on the sheet: H1, H2
Changed lines of the file:
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@@
-	)
-	(junction
-		(at 127 59.69)
-		(diameter 0)
-		(color 0 0 0 0)
 	)
 	(junction
@@
 	)
 	(junction
-		(at 118.11 69.85)
-		(diameter 0)
-		(color 0 0 0 0)
-	)
-	(junction
 		(at 144.78 130.81)
 		(diameter 0)
@@
 	)
 	(junction
-		(at 127 80.01)
-		(diameter 0)
-		(color 0 0 0 0)
-	)
-	(junction
 		(at 127 69.85)
 		(diameter 0)
@@
 	(wire
 		(pts
-			(xy 118.11 71.12) (xy 118.11 69.85)
-		)
-		(stroke
-			(width 0)
-			(type default)
-		)
-	)
-	(wire
-		(pts
 			(xy 110.49 114.3) (xy 110.49 116.84)
 		)
@@
 	(wire
 		(pts
-			(xy 118.11 69.85) (xy 118.11 68.58)
-		)
-		(stroke
-			(width 0)
-			(type default)
-		)
-	)
-	(wire
-		(pts
 			(xy 156.21 105.41) (xy 162.56 105.41)
 		)
@@
 	(wire
 		(pts
-			(xy 113.03 66.04) (xy 118.11 66.04)
-		)
-		(stroke
-			(width 0)
-			(type default)
-		)
-	)
-	(wire
-		(pts
 			(xy 115.57 114.3) (xy 115.57 120.65)
 		)
@@
 	(wire
 		(pts
-			(xy 118.11 59.69) (xy 118.11 66.04)
-		)
-		(stroke
-			(width 0)
-			(type default)
-		)
-	)
-	(wire
-		(pts
 			(xy 127 59.69) (xy 127 60.96)
 		)
@@
 	(wire
 		(pts
-			(xy 118.11 73.66) (xy 118.11 80.01)
-		)
-		(stroke
-			(width 0)
-			(type default)
-		)
-	)
-	(wire
-		(pts
 			(xy 107.95 118.11) (xy 113.03 118.11)
 		)
@@
 	(wire
 		(pts
-			(xy 113.03 68.58) (xy 118.11 68.58)
-		)
-		(stroke
-			(width 0)
-			(type default)
-		)
-	)
-	(wire
-		(pts
 			(xy 140.97 69.85) (xy 140.97 72.39)
 		)
@@
 	(wire
 		(pts
-			(xy 118.11 69.85) (xy 127 69.85)
-		)
-		(stroke
-			(width 0)
-			(type default)
-		)
-	)
-	(wire
-		(pts
 			(xy 144.78 97.79) (xy 144.78 105.41)
 		)
@@
 	(wire
 		(pts
-			(xy 113.03 73.66) (xy 118.11 73.66)
-		)
-		(stroke
-			(width 0)
-			(type default)
-		)
-	)
-	(wire
-		(pts
 			(xy 144.78 105.41) (xy 148.59 105.41)
 		)
@@
 	(wire
 		(pts
-			(xy 118.11 80.01) (xy 127 80.01)
-		)
-		(stroke
-			(width 0)
-			(type default)
-		)
-	)
-	(wire
-		(pts
 			(xy 113.03 101.6) (xy 113.03 99.06)
-		)
-		(stroke
-			(width 0)
-			(type default)
-		)
-	)
-	(wire
-		(pts
-			(xy 113.03 71.12) (xy 118.11 71.12)
-		)
-		(stroke
-			(width 0)
-			(type default)
-		)
-	)
-	(wire
-		(pts
-			(xy 118.11 59.69) (xy 127 59.69)
 		)
 		(stroke
@@
 		(on_board yes)
 		(dnp no)
-		(property "Reference" "J2"
+		(property "Reference" "J1"
 			(at 87.63 99.06 0)
 			(effects
@@
 			(project "current_converter"
 				(path "/6c1784eb-5a72-4600-8ac9-cf9d25230bce"
-					(reference "J2")
+					(reference "J1")
 					(unit 1)
 				)
@@
 	(symbol
 		(lib_id "Mechanical:MountingHole")
-		(at 87.63 73.66 0)
+		(at 101.6 73.66 0)
 		(unit 1)
 		(exclude_from_sim no)
@@
 		(fields_autoplaced yes)
 		(property "Reference" "H2"
-			(at 90.17 72.3899 0)
+			(at 104.14 72.3899 0)
 			(effects
 				(font
@@
 		)
 		(property "Value" "MountingHole"
-			(at 90.17 74.9299 0)
+			(at 104.14 74.9299 0)
 			(effects
 				(font
@@
 		)
 		(property "Footprint" "MountingHole:MountingHole_3.2mm_M3"
-			(at 87.63 73.66 0)
+			(at 101.6 73.66 0)
 			(effects
 				(font
@@
 		)
 		(property "Datasheet" "~"
-			(at 87.63 73.66 0)
+			(at 101.6 73.66 0)
 			(effects
 				(font
@@
 		)
 		(property "Description" "Mounting Hole without connection"
-			(at 87.63 73.66 0)
+			(at 101.6 73.66 0)
 			(effects
 				(font
@@
 	(symbol
 		(lib_id "Mechanical:MountingHole")
-		(at 87.63 66.04 0)
+		(at 101.6 66.04 0)
 		(unit 1)
 		(exclude_from_sim no)
@@
 		(fields_autoplaced yes)
 		(property "Reference" "H1"
-			(at 90.17 64.7699 0)
+			(at 104.14 64.7699 0)
 			(effects
 				(font
@@
 		)
 		(property "Value" "MountingHole"
-			(at 90.17 67.3099 0)
+			(at 104.14 67.3099 0)
 			(effects
 				(font
@@
 		)
 		(property "Footprint" "MountingHole:MountingHole_3.2mm_M3"
-			(at 87.63 66.04 0)
+			(at 101.6 66.04 0)
 			(effects
 				(font
@@
 		)
 		(property "Datasheet" "~"
-			(at 87.63 66.04 0)
+			(at 101.6 66.04 0)
 			(effects
 				(font
@@
 		)
 		(property "Description" "Mounting Hole without connection"
-			(at 87.63 66.04 0)
+			(at 101.6 66.04 0)
 			(effects
 				(font
@@
 		(on_board yes)
 		(dnp no)
-		(property "Reference" "J3"
+		(property "Reference" "J2"
 			(at 108.204 107.95 90)
 			(effects
@@
 			(project "current_converter"
 				(path "/6c1784eb-5a72-4600-8ac9-cf9d25230bce"
-					(reference "J3")
+					(reference "J2")
 					(unit 1)
 				)
@@
 		(on_board yes)
 		(dnp no)
-		(property "Reference" "J5"
+		(property "Reference" "J4"
 			(at 87.63 130.81 0)
 			(effects
@@
 			(project "current_converter"
 				(path "/6c1784eb-5a72-4600-8ac9-cf9d25230bce"
-					(reference "J5")
+					(reference "J4")
 					(unit 1)
 				)
@@
 		(on_board yes)
 		(dnp no)
-		(property "Reference" "J6"
+		(property "Reference" "J5"
 			(at 191.77 130.81 0)
 			(effects
@@
 			(project "current_converter"
 				(path "/6c1784eb-5a72-4600-8ac9-cf9d25230bce"
-					(reference "J6")
+					(reference "J5")
 					(unit 1)
 				)
@@
 	)
 	(symbol
-		(lib_id "Connector:Conn_01x04_Pin")
-		(at 107.95 68.58 0)
-		(unit 1)
-		(exclude_from_sim no)
-		(in_bom yes)
-		(on_board yes)
-		(dnp no)
-		(property "Reference" "J1"
-			(at 105.918 68.58 0)
-			(effects
-				(font
-					(size 1.27 1.27)
-				)
-			)
-		)
-		(property "Value" "Conn_01x04_Pin"
-			(at 108.585 63.5 0)
-			(effects
-				(font
-					(size 1.27 1.27)
-				)
-				(hide yes)
-			)
-		)
-		(property "Footprint" "Connector_PinHeader_2.54mm:PinHeader_1x04_P2.54mm_Vertical"
-			(at 107.95 68.58 0)
-			(effects
-				(font
-					(size 1.27 1.27)
-				)
-				(hide yes)
-			)
-		)
-		(property "Datasheet" "~"
-			(at 107.95 68.58 0)
-			(effects
-				(font
-					(size 1.27 1.27)
-				)
-				(hide yes)
-			)
-		)
-		(property "Description" "Generic connector, single row, 01x04, script generated"
-			(at 107.95 68.58 0)
-			(effects
-				(font
-					(size 1.27 1.27)
-				)
-				(hide yes)
-			)
-		)
-		(pin "4"
-		)
-		(pin "1"
-		)
-		(pin "3"
-		)
-		(pin "2"
-		)
-		(instances
-			(project ""
-				(path "/6c1784eb-5a72-4600-8ac9-cf9d25230bce"
-					(reference "J1")
-					(unit 1)
-				)
-			)
-		)
-	)
-	(symbol
 		(lib_id "Device:C")
 		(at 181.61 69.85 0)
@@
 		(on_board yes)
 		(dnp no)
-		(property "Reference" "J4"
+		(property "Reference" "J3"
 			(at 191.77 115.57 0)
 			(effects
@@
 			(project ""
 				(path "/6c1784eb-5a72-4600-8ac9-cf9d25230bce"
-					(reference "J4")
-					(unit 1)
-				)
+					(reference "J3")
+					(unit 1)
+				)

Commit message: Refine things
Parts:
- R1: Tolerance (none) -> 1%
- R6: value 1 -> 0.976; Tolerance 0.1% -> 1%
- U1: value OPA197xDBV -> OPA192IDBVR
Other:
- moved on the sheet: R4, R6
Changed lines of the file:
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@@
 	(generator_version "9.0")
 	(paper "A4")
+	(text_box "~25 mOhm"
+		(exclude_from_sim no)
+		(at 92.71 104.14 0)
+		(size 27.94 7.62)
+		(margins 0.9525 0.9525 0.9525 0.9525)
+		(stroke
+			(width 0)
+			(type dot)
+		)
+		(fill
+			(type none)
+		)
+		(effects
+			(font
+				(size 1.27 1.27)
+			)
+			(justify left)
+		)
+	)
 	(text_box "P_{MAX}(0805) = 1/8W\nI_{MAX}(1 Ohm) = 350 mA\nI_{MAX}(100 Ohm) = 35 mA\nI_{MAX}(10 kOhm) = 3.5 mA"
 		(exclude_from_sim no)
@@
 	)
 	(junction
-		(at 123.19 130.81)
-		(diameter 0)
-		(color 0 0 0 0)
-	)
-	(junction
 		(at 172.72 105.41)
 		(diameter 0)
@@
 	)
 	(junction
+		(at 106.68 130.81)
+		(diameter 0)
+		(color 0 0 0 0)
+	)
+	(junction
 		(at 115.57 99.06)
 		(diameter 0)
@@
 	)
 	(junction
+		(at 124.46 130.81)
+		(diameter 0)
+		(color 0 0 0 0)
+	)
+	(junction
 		(at 172.72 115.57)
+		(diameter 0)
+		(color 0 0 0 0)
+	)
+	(junction
+		(at 99.06 130.81)
 		(diameter 0)
 		(color 0 0 0 0)
@@
 	)
 	(junction
-		(at 102.87 130.81)
-		(diameter 0)
-		(color 0 0 0 0)
-	)
-	(junction
 		(at 127 69.85)
 		(diameter 0)
 		(color 0 0 0 0)
 	)
-	(junction
-		(at 107.95 130.81)
-		(diameter 0)
-		(color 0 0 0 0)
-	)
 	(wire
 		(pts
@@
 	(wire
 		(pts
-			(xy 123.19 130.81) (xy 144.78 130.81)
-		)
-		(stroke
-			(width 0)
-			(type default)
-		)
-	)
-	(wire
-		(pts
 			(xy 181.61 80.01) (xy 181.61 82.55)
 		)
@@
 	(wire
 		(pts
-			(xy 102.87 130.81) (xy 107.95 130.81)
-		)
-		(stroke
-			(width 0)
-			(type default)
-		)
-	)
-	(wire
-		(pts
-			(xy 115.57 130.81) (xy 123.19 130.81)
+			(xy 115.57 130.81) (xy 124.46 130.81)
 		)
 		(stroke
@@
 	(wire
 		(pts
-			(xy 107.95 128.27) (xy 107.95 130.81)
-		)
-		(stroke
-			(width 0)
-			(type default)
-		)
-	)
-	(wire
-		(pts
-			(xy 107.95 118.11) (xy 113.03 118.11)
+			(xy 106.68 128.27) (xy 106.68 130.81)
+		)
+		(stroke
+			(width 0)
+			(type default)
+		)
+	)
+	(wire
+		(pts
+			(xy 106.68 118.11) (xy 113.03 118.11)
 		)
 		(stroke
@@
 	(wire
 		(pts
+			(xy 99.06 130.81) (xy 106.68 130.81)
+		)
+		(stroke
+			(width 0)
+			(type default)
+		)
+	)
+	(wire
+		(pts
 			(xy 140.97 69.85) (xy 140.97 72.39)
 		)
@@
 	(wire
 		(pts
-			(xy 123.19 118.11) (xy 123.19 120.65)
+			(xy 124.46 118.11) (xy 124.46 120.65)
 		)
 		(stroke
@@
 	(wire
 		(pts
-			(xy 118.11 118.11) (xy 123.19 118.11)
+			(xy 118.11 118.11) (xy 124.46 118.11)
 		)
 		(stroke
@@
 	(wire
 		(pts
-			(xy 93.98 130.81) (xy 102.87 130.81)
-		)
-		(stroke
-			(width 0)
-			(type default)
-		)
-	)
-	(wire
-		(pts
-			(xy 123.19 128.27) (xy 123.19 130.81)
+			(xy 93.98 130.81) (xy 99.06 130.81)
+		)
+		(stroke
+			(width 0)
+			(type default)
+		)
+	)
+	(wire
+		(pts
+			(xy 124.46 128.27) (xy 124.46 130.81)
 		)
 		(stroke
@@
 	(wire
 		(pts
-			(xy 107.95 130.81) (xy 115.57 130.81)
-		)
-		(stroke
-			(width 0)
-			(type default)
-		)
-	)
-	(wire
-		(pts
 			(xy 170.18 105.41) (xy 172.72 105.41)
 		)
@@
 	(wire
 		(pts
-			(xy 102.87 116.84) (xy 102.87 130.81)
+			(xy 106.68 130.81) (xy 115.57 130.81)
+		)
+		(stroke
+			(width 0)
+			(type default)
+		)
+	)
+	(wire
+		(pts
+			(xy 99.06 116.84) (xy 99.06 130.81)
 		)
 		(stroke
@@
 	(wire
 		(pts
-			(xy 107.95 120.65) (xy 107.95 118.11)
+			(xy 106.68 120.65) (xy 106.68 118.11)
 		)
 		(stroke
@@
 	(wire
 		(pts
-			(xy 110.49 116.84) (xy 102.87 116.84)
+			(xy 110.49 116.84) (xy 99.06 116.84)
+		)
+		(stroke
+			(width 0)
+			(type default)
+		)
+	)
+	(wire
+		(pts
+			(xy 124.46 130.81) (xy 144.78 130.81)
 		)
 		(stroke
@@
 	(symbol
 		(lib_id "Device:R")
-		(at 107.95 124.46 180)
+		(at 106.68 124.46 180)
 		(unit 1)
 		(exclude_from_sim no)
@@
 		(dnp no)
 		(property "Reference" "R4"
-			(at 109.22 123.952 0)
+			(at 107.95 122.682 0)
 			(effects
 				(font
@@
 		)
 		(property "Value" "10k"
-			(at 109.22 125.73 0)
+			(at 107.95 124.46 0)
 			(effects
 				(font
@@
 		)
 		(property "Footprint" "Resistor_SMD:R_0805_2012Metric_Pad1.20x1.40mm_HandSolder"
-			(at 109.728 124.46 90)
+			(at 108.458 124.46 90)
 			(effects
 				(font
@@
 		)
 		(property "Datasheet" "~"
-			(at 107.95 124.46 0)
+			(at 106.68 124.46 0)
 			(effects
 				(font
@@
 		)
 		(property "Description" "Resistor"
-			(at 107.95 124.46 0)
+			(at 106.68 124.46 0)
 			(effects
 				(font
@@
 		)
 		(property "Tolerance" "0.05%"
-			(at 111.252 128.27 0)
+			(at 110.998 126.238 0)
 			(effects
 				(font
@@
 			)
 		)
-		(property "Value" "OPA197xDBV"
+		(property "Value" "OPA192IDBVR"
 			(at 167.894 120.142 0)
 			(effects
@@
 		(dnp no)
 		(property "Reference" "R5"
-			(at 116.84 123.952 0)
+			(at 116.84 122.682 0)
 			(effects
 				(font
@@
 		)
 		(property "Value" "100"
-			(at 116.84 125.73 0)
+			(at 116.84 124.46 0)
 			(effects
 				(font
@@
 		)
 		(property "Tolerance" "0.05%"
-			(at 118.872 128.27 0)
+			(at 119.888 126.238 0)
 			(effects
 				(font
@@
 	(symbol
 		(lib_id "Device:R")
-		(at 123.19 124.46 180)
+		(at 124.46 124.46 180)
 		(unit 1)
 		(exclude_from_sim no)
@@
 		(dnp no)
 		(property "Reference" "R6"
-			(at 124.46 123.952 0)
+			(at 125.73 122.682 0)
 			(effects
 				(font
@@
 			)
 		)
-		(property "Value" "1"
-			(at 124.46 125.73 0)
+		(property "Value" "0.976"
+			(at 125.73 124.46 0)
 			(effects
 				(font
@@
 		)
 		(property "Footprint" "Resistor_SMD:R_0805_2012Metric_Pad1.20x1.40mm_HandSolder"
-			(at 124.968 124.46 90)
+			(at 126.238 124.46 90)
 			(effects
 				(font
@@
 		)
 		(property "Datasheet" "~"
-			(at 123.19 124.46 0)
+			(at 124.46 124.46 0)
 			(effects
 				(font
@@
 		)
 		(property "Description" "Resistor"
-			(at 123.19 124.46 0)
-			(effects
-				(font
-					(size 1.27 1.27)
-				)
-				(hide yes)
-			)
-		)
-		(property "Tolerance" "0.1%"
-			(at 126.492 128.27 0)
+			(at 124.46 124.46 0)
+			(effects
+				(font
+					(size 1.27 1.27)
+				)
+				(hide yes)
+			)
+		)
+		(property "Tolerance" "1%"
+			(at 127.254 126.238 0)
 			(effects
 				(font
@@
 		(dnp no)
 		(property "Reference" "R7"
-			(at 146.05 123.19 0)
+			(at 146.05 122.682 0)
 			(effects
 				(font
@@
 		)
 		(property "Value" "1k"
-			(at 146.05 125.73 0)
+			(at 146.05 124.46 0)
 			(effects
 				(font
@@
 		)
 		(property "Tolerance" "0.05%"
-			(at 148.082 128.27 0)
+			(at 149.098 126.238 0)
 			(effects
 				(font
@@
 		(dnp no)
 		(property "Reference" "R1"
-			(at 134.62 104.14 0)
+			(at 134.62 103.632 0)
 			(effects
 				(font
@@
 		)
 		(property "Value" "270"
-			(at 134.62 106.68 0)
+			(at 134.62 105.41 0)
 			(effects
 				(font
@@
 				)
 				(hide yes)
+			)
+		)
+		(property "Tolerance" "1%"
+			(at 136.144 107.188 0)
+			(effects
+				(font
+					(size 1.27 1.27)
+				)
 			)
 		)
@@
 		(dnp no)
 		(property "Reference" "C1"
+			(at 185.928 68.834 0)
+			(effects
+				(font
+					(size 1.27 1.27)
+				)
+			)
+		)
+		(property "Value" "1uF"
 			(at 186.436 70.866 0)
 			(effects
 				(font
-					(size 1.27 1.27)
-				)
-			)
-		)
-		(property "Value" "1uF"
-			(at 186.436 68.834 0)
-			(effects
-				(font
